File: electronics/PDB/miranda-pdb.kicad_pcb (KiCad board)
At the start: 2 copper layers, 23 parts, among them IC1 MP2315GJ-Z, IC2 MP2315GJ-Z, U1 INA180A3

Commit message: finished pdb
Parts:
- added C1: 0.1uf, Capacitor_SMD:C_0805_2012Metric, F.Cu at (97.2, 119.7)
- added C10: 0.1uf, Capacitor_SMD:C_0805_2012Metric, F.Cu at (114.3, 119.7)
- added C11: 0.1uf, Capacitor_SMD:C_0805_2012Metric, F.Cu at (106.5, 109.7)
- added C2: 22uf, Capacitor_SMD:C_0805_2012Metric, F.Cu at (97.7, 125.5)
- added C3: 0.1uf, Capacitor_SMD:C_0805_2012Metric, F.Cu at (95.1, 115.5)
- added C4: 22uf, Capacitor_SMD:C_0805_2012Metric, F.Cu at (97.7, 123.5)
- added C5: 22uf, Capacitor_SMD:C_0805_2012Metric, F.Cu at (87.1, 115.5)
- added C6: 22uf, Capacitor_SMD:C_0805_2012Metric, F.Cu at (104.3, 115.7)
- added C7: 0.1uf, Capacitor_SMD:C_0805_2012Metric, F.Cu at (112.3, 115.7)
- added C8: 22uf, Capacitor_SMD:C_0805_2012Metric, F.Cu at (114.9, 125.4)
- added C9: 22uf, Capacitor_SMD:C_0805_2012Metric, F.Cu at (114.9, 123.4)
- added J1: Conn_01x02, Connector:solder pad, F.Cu at (114.9, 107.7)
- added J10: Conn_01x03, Connector_AMASS:MR30PW-FB, F.Cu at (90.3, 91.2)
- added J11: Conn_01x03, Connector_AMASS:MR30PW-FB, F.Cu at (107.3, 91.2)
- added J16: Conn_02x04_Odd_Even, Connector_PinHeader_2.54mm:PinHeader_2x04_P2.54mm_Horizontal, F.Cu at (109.0, 129.5)
- added J2: Conn_02x04_Odd_Even, Connector_PinHeader_2.54mm:PinHeader_2x04_P2.54mm_Horizontal, F.Cu at (95.9, 129.5)
- added J3: Conn_02x03_Odd_Even, Connector_PinHeader_2.54mm:PinHeader_2x03_P2.54mm_Horizontal, F.Cu at (83.8, 124.7)
- added J4: Conn_01x02, Connector:solder pad, F.Cu at (83.1, 107.4)
- R10, R3, R6, R7: moved to B.Cu
- moved R18 48.2 mm to (86.6, 124.7), turned to 90 degrees
- moved R6 43.4 mm to (89.3, 115.4), turned to 90 degrees
- moved R17 42.0 mm to (103.8, 124.7), turned to 90 degrees
- moved L1 41.1 mm to (91.8, 122.3), turned to -90 degrees
- moved R1 41.0 mm to (89.3, 115.4), turned to -90 degrees
- moved R11 40.6 mm to (116.6, 119.9), turned to 90 degrees
- moved D4 39.1 mm to (86.6, 120.9), turned to -90 degrees
- moved R2 35.1 mm to (97.3, 115.4), turned to -90 degrees
- moved R7 34.0 mm to (106.5, 115.5), turned to -90 degrees
- moved R12 33.4 mm to (116.6, 115.5), turned to 90 degrees
- moved R4 32.7 mm to (99.6, 119.6), turned to 90 degrees
- moved R3 32.3 mm to (97.3, 115.4), turned to -90 degrees
- moved L2 31.8 mm to (109.0, 122.3), turned to -90 degrees
- moved R8 31.2 mm to (106.4, 115.5), turned to -90 degrees
- moved D3 30.1 mm to (103.8, 120.7), turned to -90 degrees
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Connections:
- IC1 pad 7: +BATT -> Net-(IC1-VCC)
- IC2 pad 7: +BATT -> Net-(IC2-VCC)
- L2 pad 2: +5V -> +12V
- R11 pad 1: +5V -> +12V
- R7 pad 1: +BATT -> Net-(IC2-EN/SYNC)
- R7 pad 2: Net-(IC2-EN/SYNC) -> +BATT
Routing:
- net /M2_SIGNAL: track 0.00 -> 46.6 mm, vias 0 -> 1
- net /Current sense: track 0.00 -> 43.8 mm, vias 0 -> 1
- net /M1_SIGNAL: track 0.00 -> 29.3 mm
- net +5V: track 0.00 -> 15.3 mm
- net GND: track 0.00 -> 10.6 mm, vias 0 -> 35
- net Net-(IC1-FB): track 0.00 -> 8.89 mm, vias 0 -> 1
- net Net-(IC2-FB): track 0.00 -> 8.72 mm, vias 0 -> 1
- net Net-(R10-Pad2): track 0.00 -> 6.72 mm, vias 0 -> 1
- net Net-(IC2-VCC): track 0.00 -> 5.46 mm
- net Net-(IC2-BST): track 0.00 -> 5.45 mm
- net Net-(R3-Pad2): track 0.00 -> 5.40 mm, vias 0 -> 1
- net Net-(IC1-BST): track 0.00 -> 5.36 mm
- net Net-(IC1-VCC): track 0.00 -> 5.24 mm
- net Net-(IC1-EN/SYNC): track 0.00 -> 4.51 mm, vias 0 -> 1
- net Net-(IC2-EN/SYNC): track 0.00 -> 4.49 mm, vias 0 -> 1
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- added copper zone on F.Cu, net +12V
- added copper zone on F.Cu, net +5V
- added copper zone on B.Cu, net +BATT
- added copper zone on F.Cu, net +BATT
- added copper zone on B.Cu, net GND
- added copper zone on F.Cu, net GND
- added copper zone on F.Cu, net Net-(IC1-AAM)
- added copper zone on F.Cu, net Net-(IC1-SW)
- added copper zone on F.Cu, net Net-(IC2-AAM)
- added copper zone on F.Cu, net Net-(IC2-SW)
- added copper zone on F.Cu, net Net-(J1-Pin_2)
Other:
- board outline added: 38.7 x 46.1 mm
- board text added: "+12V"
- board text added: "+5V"
- board text added: "2-4S IN"
- board text added: "2-4S OUT"
- board text added: "CUR"
- board text added: "GND"
- board text added: "M1"
- board text added: "M2"
