File: electronics/PDB/miranda-pdb.kicad_sch (KiCad schematic)
At the start: 48 parts, among them IC1 MP2315GJ-Z, IC2 MP2315GJ-Z, J1 Conn_01x02, J10 Conn_01x03, J11 Conn_01x03, J12 Conn_01x03, J13 Conn_01x03, J14 Conn_01x03, J2 Conn_01x03, J3 Conn_01x03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

Commit message: finished pdb
Parts:
- removed J12, J13, J14, J2, J3, J4, J5, J6, J7, J8, J9: Conn_01x03, symbol Connector_Generic:Conn_01x03
- added J16, J2: Conn_02x04_Odd_Even, Connector_PinHeader_2.54mm:PinHeader_2x04_P2.54mm_Horizontal, symbol Connector_Generic:Conn_02x04_Odd_Even
- added J3: Conn_02x03_Odd_Even, Connector_PinHeader_2.54mm:PinHeader_2x03_P2.54mm_Horizontal, symbol Connector_Generic:Conn_02x03_Odd_Even
- added J4: Conn_01x02, Connector:solder pad, symbol Connector_Generic:Conn_01x02
- C1, C10, C11, C2, C3, C4, C5, C6, C7, C8, C9: footprint (none) -> Capacitor_SMD:C_0805_2012Metric
- IC1, IC2: footprint SOT65P280X100-8N -> SamacSys_Parts:SOT65P280X100-8N
- J1: footprint (none) -> Connector:solder pad
- J10, J11: footprint (none) -> Connector_AMASS:MR30PW-FB
Connections:
- net +12V: now also C8.2, C9.2, L2.2, R11.1, J16.1 (Pin_1), J16.3 (Pin_3), J16.5 (Pin_5), J16.7 (Pin_7)
- net +5V: now also J2.1 (Pin_1), J2.3 (Pin_3), J2.5 (Pin_5), J2.7 (Pin_7); no longer C8.2, C9.2, L2.2, R11.1
- net +BATT: now also R7.2, J4.2 (Pin_2); no longer C3.2, C7.2, IC1.7 (VCC), IC2.7 (VCC), R7.1
- net Current sense: now also J3.2 (Pin_2)
- net GND: now also J16.2 (Pin_2), J16.4 (Pin_4), J16.6 (Pin_6), J16.8 (Pin_8), J2.2 (Pin_2), J2.4 (Pin_4), J2.6 (Pin_6), J2.8 (Pin_8), J3.1 (Pin_1), J3.3 (Pin_3), J3.5 (Pin_5), J4.1 (Pin_1)
- net M1_SIGNAL: now also J3.6 (Pin_6)
- net M2_SIGNAL: now also J3.4 (Pin_4)
- net at IC2.6 (EN/SYNC): now also R7.1; no longer R7.2
- new net: C7.2, IC2.7 (VCC)
- new net: C3.2, IC1.7 (VCC)
Other:
- moved on the sheet: C1, C10, C3, C7, IC1, IC2, L1, L2, R1, R10, R11, R12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
